File: kicad/PiFinder_v3/PiFinder_smt.kicad_pcb (KiCad board)
At the start: 2 copper layers, 93.8 x 64.2 mm, 54 parts, among them J1 Raspberry_Pi_2_3, J2 display, J4 GPS Module, Q1 Q_NPN_EBC, SW0 SW_Push_Dual, SW1 SW_Push_Dual, SW2 SW_Push_Dual, SW3 SW_Push_Dual, SW4 SW_Push_Dual, SW5 SW_Push_Dual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

Commit message: Change LED footprint, cleanup silkscreen
Parts:
- D1, D10, D11, D12, D13, D14, D15, D16, D17, D2, D3, D4, D5, D6, D7, D8, D9: footprint LED_SMD:LED_1210_3225Metric -> LED_SMD:LED_1206_3216Metric
Other:
- board text added: "DIY v3.1 SMT"
- board text removed: "DIY v3 SMT"
